Commit message: Update from ecoreset branch

File: hrr_ee_tools/description/screwdriver.xacro (robot description, xacro)
@@ -35,5 +35,5 @@
     </joint>
     <joint name="${prefix}screwdriver_body_tip" type="fixed">
-      <origin xyz="-0.035 0.0 0.224" rpy="0 0 0"/>
+      <origin xyz="-0.035 0.0 0.1583" rpy="0 0 0"/>
       <parent link="${prefix}screwdriver_body"/>
       <child link="${prefix}screwdriver_tip"/>

File: hrr_ee_tools/description/toolchanger.xacro (robot description, xacro)
@@ -68,5 +68,5 @@
     </joint>
     <joint name="${prefix}toolchanger_B_tip" type="fixed">
-      <origin xyz="0 0.0 0.0215" rpy="0 0 0.0"/>
+      <origin xyz="0 0.0 0.0215" rpy="0 0 1.5707963267948966"/>
       <parent link="${prefix}toolchanger_body_B"/>
       <child link="${prefix}toolchanger_connect"/>

File: hrr_ee_tools/description/vacuum.xacro (robot description, xacro)
@@ -40,5 +40,5 @@
     </joint>
     <joint name="${prefix}vacuum_body_tip_2" type="fixed">
-      <origin xyz="-0.003 -0.0525 0.08568" rpy="0 0 0"/>
+      <origin xyz="0 -0.0525 0.11568" rpy="0 0 0"/> <!---0.003 -0.0525 0.08568-->
       <parent link="${prefix}vacuum_body"/>
       <child link="${prefix}vacuum_tip_2"/>
